Commit message: .

File: prodigimover-small_description/urdf/prodigimover.urdf (robot description, URDF)
Before this commit: robot prodigimover, 9 links, 8 joints
Links:
- link base_link: geometry collision mesh filename=package://prodigimover_description/meshes/Base_Link.STL; visual mesh filename=package://prodigimover_description/meshes/Base_Link.STL

Commit message: ..

File: prodigimover-small_description/urdf/prodigimover.urdf (robot description, URDF)
Before this commit: robot prodigimover, 9 links, 8 joints
Links:
- link base_link: geometry collision mesh filename=package://prodigimover-small_description/meshes/base_link.S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; visual mesh filename=package://prodigimover-small_description/meshes/base_link.S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
- link camera_link: geometry collision mesh filename=package://prodigimover_description/meshes/ProdigiMover_Zedm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 scale=0.001 0.001 0.001; visual mesh filename=package://prodigimover-small_description/meshes/ProdigiMove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 scale=0.001 0.001 0.001
- link laser_link: geometry collision mesh filename=package://prodigimover-small_description/meshes/ProdigiMove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 scale=0.001 0.001 0.001; visual mesh filename=package://prodigimover-small_description/meshes/ProdigiMove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 scale=0.001 0.001 0.001
- link wheel_front_left_link: geometry collision mesh filename=package://prodigimover-small_description/meshes/front_left_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; visual mesh filename=package://prodigimover-small_description/meshes/front_left_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
- link wheel_front_right_link: geometry collision mesh filename=package://prodigimover-small_description/meshes/front_right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; visual mesh filename=package://prodigimover-small_description/meshes/front_right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
- link wheel_rear_left_link: geometry collision mesh filename=package://prodigimover-small_description/meshes/back_left_w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; visual mesh filename=package://prodigimover-small_description/meshes/back_left_w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
- link wheel_rear_right_link: geometry collision mesh filename=package://prodigimover-small_description/meshes/back_right_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; visual mesh filename=package://prodigimover-small_description/meshes/back_right_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
