Commit message: .

File: prodigimover-small_description/urdf/prodigimover.urdf.xacro (robot description, xacro)
@@ -1,4 +1,6 @@
 <?xml version="1.0"?>
 <robot name="prodigimover" xmlns:xacro="http://www.ros.org/wiki/xacro">
+    <xacro:include filename="$(find prodigimover-small_description)/urdf/prodigimover_gazebo.xacro" />
+    <xacro:prodigimover_gazebo />
     <link name="robot_footprint"/>
     <link name="imu_link"/>
@@ -65,5 +67,5 @@
     </link>
     <joint name="wheel_front_right_joint" type="continuous">
-        <origin xyz="0.08 -0.0845 -0.0389" rpy="-1.5703 0 3.14159"/>
+        <origin xyz="0.08 -0.0845 -0.0389" rpy="1.5707 0 3.1415"/>
         <parent link="base_link"/>
         <child link="wheel_front_right_link"/>
@@ -95,5 +97,5 @@
     </link>
     <joint name="wheel_front_left_joint" type="continuous">
-        <origin xyz="0.08 0.084492 -0.0389" rpy="1.5703 0 0"/>
+        <origin xyz="0.08 0.084492 -0.0389" rpy="1.5707 0 3.1415"/>
         <parent link="base_link"/>
         <child link="wheel_front_left_link"/>
@@ -125,5 +127,5 @@
     </link>
     <joint name="wheel_rear_right_joint" type="continuous">
-        <origin xyz="-0.08 -0.0845 -0.03946" rpy="-1.57 0 3.14159"/>
+        <origin xyz="-0.08 -0.0845 -0.03946" rpy="1.5707 0 3.1415"/>
         <parent link="base_link"/>
         <child link="wheel_rear_right_link"/>
@@ -155,5 +157,5 @@
     </link>
     <joint name="wheel_rear_left_joint" type="continuous">
-        <origin xyz="-0.08 0.084492 -0.03954" rpy="1.5703 0 0"/>
+        <origin xyz="-0.08 0.084492 -0.03954" rpy="1.5707 0 3.1415"/>
         <parent link="base_link"/>
         <child link="wheel_rear_left_link"/>
@@ -178,5 +180,5 @@
         </visual>
         <collision>
-            <origin xyz="0 0 0" rpy="0 0 0"/>
+            <origin xyz="0 0.045 -0.025" rpy="1.5707 0 0"/>
             <geometry>
                 <mesh filename="package://prodigimover-small_description/meshes/ProdigiMover_YDLidar_G2.stl" scale="0.001 0.001 0.001"/>
@@ -216,142 +218,3 @@
         <child link="camera_link"/>
     </joint>
-    <!-- GAZEBO PLUGINS -->
-    <gazebo reference="wheel_front_right_link">
-      <material value="Gazebo/FlatBlack"/>
-      <mu1>1.16</mu1>
-      <mu2>1.16</mu2>
-      <kp>5000000.0</kp>
-      <kd>10.0</kd>
-      <maxVel>4.0</maxVel>
-      <fdir1>0 0 0</fdir1>
-      <turnGravityOff>false</turnGravityOff>
-    </gazebo>
-    <gazebo reference="wheel_front_left_link">
-      <material value="Gazebo/FlatBlack"/>
-      <mu1>1.16</mu1>
-      <mu2>1.16</mu2>
-      <kp>5000000.0</kp>
-      <kd>10.0</kd>
-      <maxVel>4.0</maxVel>
-      <fdir1>0 0 0</fdir1>
-      <turnGravityOff>false</turnGravityOff>
-    </gazebo>
-    <gazebo reference="wheel_rear_right_link">
-      <material value="Gazebo/FlatBlack"/>
-      <mu1>1.16</mu1>
-      <mu2>1.16</mu2>
-      <kp>5000000.0</kp>
-      <kd>10.0</kd>
-      <maxVel>4.0</maxVel>
-      <fdir1>0 0 0</fdir1>
-      <turnGravityOff>false</turnGravityOff>
-    </gazebo>
-    <gazebo reference="wheel_rear_left_link">
-      <material value="Gazebo/FlatBlack"/>
-      <mu1>1.16</mu1>
-      <mu2>1.16</mu2>
-      <kp>5000000.0</kp>
-      <kd>10.0</kd>
-      <maxVel>4.0</maxVel>
-      <fdir1>0 0 0</fdir1>
-      <turnGravityOff>false</turnGravityOff>
-    </gazebo>
-            <!-- Transmission is important to link the joints and the controller -->
-        <transmission name="wheel_front_right_trans">
-            <type>transmission_interface/SimpleTransmission</type>
-            <joint name="wheel_front_right_joint"/>
-            <actuator name="wheel_front_right_joint_motor">
-                <hardwareInterface>EffortJointInterface</hardwareInterface>
-                <mechanicalReduction>1</mechanicalReduction>
-            </actuator>
-        </transmission>
-        <transmission name="wheel_front_left_trans">
-            <type>transmission_interface/SimpleTransmission</type>
-            <joint name="wheel_front_left_joint"/>
-            <actuator name="wheel_front_left_joint_motor">
-                <hardwareInterface>EffortJointInterface</hardwareInterface>
-                <mechanicalReduction>1</mechanicalReduction>
-            </actuator>
-        </transmission>
-        <transmission name="wheel_rear_right_trans">
-            <type>transmission_interface/SimpleTransmission</type>
-            <joint name="wheel_rear_right_joint"/>
-            <actuator name="wheel_rear_right_joint_motor">
-                <hardwareInterface>EffortJointInterface</hardwareInterface>
-                <mechanicalReduction>1</mechanicalReduction>
-            </actuator>
-        </transmission>
-        <transmission name="wheel_rear_left_trans">
-            <type>transmission_interface/SimpleTransmission</type>
-            <joint name="wheel_rear_left_joint"/>
-            <actuator name="wheel_rear_left_joint_motor">
-                <hardwareInterface>EffortJointInterface</hardwareInterface>
-                <mechanicalReduction>1</mechanicalReduction>
-            </actuator>
-        </transmission>
-        <gazebo reference="laser_link" >
-            <material value="Gazebo/Red" />
-            <sensor type="ray" name="lidar" >
-                <tf_prefix>prodigimover</tf_prefix>
-                <pose>0 0 0 0 0 0</pose>
-                <always_on>true</always_on>
-                <visualize>false</visualize>
-                <update_rate>10</update_rate>
-                <ray>
-                    <scan>
-                        <horizontal>
-                            <samples>720</samples>
-                            <resolution>1</resolution>
-                            <min_angle>-3.141592</min_angle>
-                            <max_angle>3.141592</max_angle>
-                        </horizontal>
-                    </scan>
-                    <range>
-                        <min>0.12</min>
-                        <max>16.0</max>
-                        <resolution>0.03</resolution>
-                    </range>
-                    <noise>
-                        <type>gaussian</type>
-                        <mean>0.0</mean>
-                        <stddev>0.01</stddev>
-                    </noise>
-                </ray>
-                <plugin name="laser_scan_plugin" filename="libgazebo_ros_laser.so" >
-                    <output_type>sensor_msgs/LaserScan</output_type>
-                    <robotNamespace>prodigimover</robotNamespace>
-                    <topicName>scan</topicName>
-                    <frameName>laser_link</frameName>
-                </plugin>
-            </sensor>
-        </gazebo>
-        <!-- Skid Steer Drive -->
-        <gazebo>
-            <plugin name="skid_steer_drive_controller" filename="libgazebo_ros_skid_steer_drive.so">
-                <updateRate>5.0</updateRate>
-                <robotNamespace>prodigimover</robotNamespace>
-                <leftFrontJoint>wheel_front_left_joint</leftFrontJoint>
-                <rightFrontJoint>wheel_front_right_joint</rightFrontJoint>
-                <leftRearJoint>wheel_rear_left_joint</leftRearJoint>
-                <rightRearJoint>wheel_rear_right_joint</rightRearJoint>
-                <wheelSeparation>0.584</wheelSeparation>
-                <wheelDiameter>0.26</wheelDiameter>
-                <robotBaseFrame>robot_footprint</robotBaseFrame>
-                <torque>50</torque>
-                <MaxForce>5.0</MaxForce>
-                <topicName>cmd_vel</topicName>
-                <commandTopic>cmd_vel</commandTopic>
-                <odometryTopic>odom</odometryTopic>
-                <odometryFrame>odom</odometryFrame>
-                <topic_name_joint>joint</topic_name_joint>
-                <broadcastTF>true</broadcastTF>
-                <publish_odom>true</publish_odom>
-                <publish_odom_tf>false</publish_odom_tf>
-                <publish_wheel_tf>true</publish_wheel_tf>
-                <covariance_x>0.0001</covariance_x>
-                <covariance_y>0.0001</covariance_y>
-                <covariance_roll>0.01</covariance_roll>
-                <covariance_yaw>0.01</covariance_yaw>
-            </plugin>
-        </gazebo>
 </robot>
